File: ms1.brd (EAGLE design)
At the start: 160 x 100 mm, 149 parts, among them IC1 MAX3232EUE, IC2 MAX3380EEUP, J1 POWERPOLE_POWER25A, J10 Radio, J11 A3, J12 A4, J13 A5, J14 A6, J15 A7, J16 D1, J17 D2, J18 D3, J19 D4, J2 ON, J20 D5, J21 D6, J22 D7, J3 LED-EN, J4 RS232, J5 RS485, J6 A1, J7 I2C, J8 A2, J9 TTL_SERIAL, Q1 DMG6602SVT, Q2 DMG6602SVT, Q3 DMG6602SVT, Q4 DMG6602SVT, U1 LT1934ES6TRMPBF, U2 LT1934ES6TRMPBF, U3 DS3231SN, U4 ISL3179EIBZ, X1 KUSBVX-BS1N

Commit message: now uses correct serial buffer
Parts:
- removed C17, C18, C22, C23: 0.1uF, resistor:A/3216-18W
- removed C26: 100nF, resistor:C0805
- removed IC2: MAX3380EEUP, basestation:TSSOP20
- removed J11: A3, farnell-parts:4-MOLEX
- removed J12: A4, farnell-parts:4-MOLEX
- removed J13: A5, farnell-parts:4-MOLEX
- removed J14: A6, farnell-parts:4-MOLEX
- removed J15: A7, farnell-parts:4-MOLEX
- removed J16: D1, farnell-parts:4-MOLEX
- removed J17: D2, farnell-parts:4-MOLEX
- removed J18: D3, farnell-parts:4-MOLEX
- removed J19: D4, farnell-parts:4-MOLEX
- removed J20: D5, farnell-parts:4-MOLEX
- removed J21: D6, farnell-parts:4-MOLEX
- removed J22: D7, farnell-parts:4-MOLEX
- removed J6: A1, farnell-parts:4-MOLEX
- removed J8: A2, farnell-parts:4-MOLEX
- removed JP10: D2, pinhead:1X04
- removed JP11: D3, pinhead:1X04
- removed JP12: D4, pinhead:1X04
- removed JP13: D5, pinhead:1X04
- removed JP14: D6, pinhead:1X04
- removed JP15: D7, pinhead:1X04
- removed JP3: A2, pinhead:1X04
- removed JP4: A3, pinhead:1X04
- removed JP5: A4, pinhead:1X04
- removed JP6: A5, pinhead:1X04
- removed JP7: A6, pinhead:1X04
- removed JP9: D1, pinhead:1X04
- removed UART1_RX, UART1_TX: TPB2,54, testpad:B2,54
- added R7: 47K, resistor:R0805
- added U$4: TXS0108E, basestation:TSSOP20
- JP2: value A1 -> (none); device pinhead:1X04 -> jumper:JP2
- moved JP2 217.9 mm to (-232.4, -1.02), turned to 0 degrees
Connections:
- removed net A_GND: J11.1, J12.1, J13.1, J14.1, J15.1, J6.1, J8.1
- removed net HADC_1: J6.2, JP2.4
- removed net HADC_2: J8.2, JP3.4
- removed net HADC_3: J11.2, JP4.4
- removed net HADC_4: J12.2, JP5.4
- removed net HADC_5: J13.2, JP6.4
- removed net HADC_6: J14.2, JP7.4
- removed net HADC_7: J15.2
- removed net HDIO_1: J16.2, JP9.4
- removed net HDIO_2: J17.2, JP10.4
- removed net HDIO_3: J18.2, JP11.4
- removed net HDIO_4: J19.2, JP12.4
- removed net HDIO_5: J20.2, JP13.4
- removed net HDIO_6: J21.2, JP14.4
- removed net HDIO_7: J22.2, JP15.4
- removed net N$64: C17.-, IC2.3
- removed net N$82: C18.+, IC2.4
- removed net N$83: C18.-, IC2.5
- removed net N$84: C22.-, IC2.6
- removed net N$9: C23.+, IC2.2
- removed net WADC_1: JP2.2
- removed net WADC_2: JP3.2
- removed net WADC_3: JP4.2
- removed net WADC_4: JP5.2
- removed net WADC_5: JP6.2
- removed net WADC_6: JP7.2
- removed net WDIO_1: JP9.2
- removed net WDIO_2: JP10.2
- removed net WDIO_3: JP11.2
- removed net WDIO_4: JP12.2
- removed net WDIO_5: JP13.2
- removed net WDIO_6: JP14.2
- removed net WDIO_7: JP15.2
- new net 232_RX: IC1.12, U$4.3
- new net 232_TX: IC1.11, U$4.5
- new net 323_3V3: C19.2, IC1.16, JP2.3
- new net 485_3V3: C14.1, JP2.1, R32.2, U4.8
- new net 485_RX: U$4.1, U4.1
- new net 485_TX: U$4.4, U4.4
- net ADC_1: no longer JP2.3
- net ADC_2: no longer JP3.3
- net ADC_3: no longer JP4.3
- net ADC_4: no longer JP5.3
- net ADC_5: no longer JP6.3
- net ADC_6: no longer JP7.3
- net DIO_1: no longer JP9.3
- net DIO_2: no longer JP10.3
- net DIO_3: no longer JP11.3, U$2.C46
- net DIO_4: no longer JP12.3
- net DIO_5: no longer JP13.3, U$2.C45
- net DIO_6: no longer JP14.3, U$2.C49
- net DIO_7: no longer JP15.3
- net GND: now also U$4.11; no longer C22.+, C23.-, C26.2, IC2.18, J16.1, J17.1, J18.1, J19.1, J20.1, J21.1, J22.1
- net N$8: now also R7.1, U$4.10; no longer C17.+, IC2.1
- net SENSE_3V3: now also JP2.2, R7.2, U$4.2; no longer C14.1, C19.2, IC1.16, IC2.13, J11.3, J12.3, J13.3, J14.3, J15.3, J16.3, J17.3, J18.3, J19.3, J20.3, J21.3, J22.3, J6.3, J8.3, JP10.1, JP11.1, JP12.1, JP13.1, JP14.1, JP15.1, JP2.1, JP3.1, JP4.1, JP5.1, JP6.1, JP7.1, JP9.1, R32.2, U4.8
- net SENSE_5V: no longer J11.4, J12.4, J13.4, J14.4, J15.4, J16.4, J17.4, J18.4, J19.4, J20.4, J21.4, J22.4, J6.4, J8.4
- net UART1_RX: now also U$4.18, U$4.20; no longer IC2.9, UART1_RX.TP
- net UART1_RX_BUF: no longer IC1.12, IC2.16, U4.1
- net UART1_TX: now also U$4.16, U$4.17; no longer IC2.8, UART1_TX.TP
- net UART1_TX_BUF: no longer IC1.11, IC2.17, U4.4
- net VCC_3V3: now also U$4.19; no longer C26.1, IC2.12, IC2.19, IC2.20
Routing:
- net SENSE_3V3: track 305.2 -> 297.9 mm
- net N$84: track 6.42 -> 0.00 mm
- net N$83: track 6.34 -> 0.00 mm
- net 485_3V3: track 0.00 -> 5.39 mm
- net N$82: track 4.75 -> 0.00 mm
- net N$8: track 3.69 -> 0.00 mm
- net N$9: track 3.50 -> 0.00 mm
- net N$64: track 2.98 -> 0.00 mm
- net 323_3V3: track 0.00 -> 1.98 mm

Commit message: now has: * rain gauge input * 2 digital io * 2 analog io * poly fuses
Parts:
- removed LED3: D3, led:CHIP-LED0805
- removed LED4: D4, led:CHIP-LED0805
- removed LED5: D5, led:CHIP-LED0805
- removed LED6: D6, led:CHIP-LED0805
- removed R13, R15, R16, R17: 56, resistor:R0805
- added J11, J12: 4-PIN-MOLEX, farnell-parts:4-MOLEX
- added J13, J14, J8: ADC2, farnell-parts:3-MOLEX
- added J6: ADC1, farnell-parts:3-MOLEX
- added R31: 100K, resistor:R0805
- added U$5, U$6, U$7: MCF0805, farnell-parts:0805
- J5: value RS485 -> 2-PIN-MOLEX; device farnell-parts:5-MOLEX -> farnell-parts:2-MOLEX
- moved J5 145.5 mm to (-256.7, -55.0)
Connections:
- removed net ADC_3: U$2.A5
- removed net ADC_4: U$2.A7
- removed net ADC_5: U$2.A10
- removed net ADC_6: U$2.A8
- removed net DIO_3: R13.2
- removed net DIO_4: R15.2
- removed net DIO_5: R16.2
- removed net DIO_6: R17.2
- removed net DIO_7: R18.2
- removed net N$11: LED6.A, R17.1
- removed net N$18: LED4.A, R15.1
- removed net N$19: LED3.A, R13.1
- removed net N$21: LED5.A, R16.1
- removed net UART1_RX_BUF: J9.2
- removed net UART1_TX_BUF: J9.3
- removed net VCC-3V: U$2.A14, U$2.A4
- new net ADC_3V3: U$2.A14, U$2.A4
- new net N$17: J12.4, U$6.1
- new net N$26: J5.1, U$7.1
- new net N$9: J11.4, U$5.1
- new net RAIN: J5.2, R18.2, R31.2, U$2.C49
- new net TTL_RX: J9.2, U$4.4
- new net TTL_TX: J9.3, U$4.7
- net 232_TX: now also U$4.6; no longer U$4.5
- net 485_TX: now also U$4.5; no longer U$4.4
- net ADC_1: now also J6.2
- net ADC_2: now also J8.2
- net AGND: now also J6.3, J8.3
- net DIO_1: now also J13.2, U$2.C46, U$2.C51
- net DIO_2: now also J14.2
- net GND: now also J11.1, J12.1, J13.3, J14.3, R31.1; no longer J5.1
- net LGND: no longer LED3.C, LED4.C, LED5.C, LED6.C
- net RS232_RXD: now also J12.2
- net RS232_TXD: now also J12.3
- net RS485_N: now also J11.2; no longer J5.2
- net RS485_P: now also J11.3; no longer J5.3
- net SENSE_3V3: now also J13.1, J14.1, J6.1, J8.1; no longer J5.4
- net SENSE_5V: now also U$5.2, U$6.2; no longer J5.5
- net UART1_RX: now also U$4.17
- net UART1_TX: now also U$4.14, U$4.15; no longer U$4.17
- net VCC_3V3: now also U$7.2
